Commit message: [urdf] Fix path to wing.stl.

File: urdf/airfoil.urdf (robot description, URDF)
Before this commit: robot Airfoil, 337 links, 336 joints
Links:
- link base_link: geometry collision mesh filename=package://agimus_demos/tiago/deburring/meshes/wing.stl scale=0.001 0.001 0.001; visual mesh filename=package://agimus_demos/tiago/deburring/meshes/wing.stl scale=0.001 0.001 0.001
